Commit message: 修复仿真小车里程计数据

File: src/laser-tag_nav_description/urdf/robot.gazebo.xacro (robot description, xacro)
@@ -1,5 +1,5 @@
 <?xml version="1.0"?>
 <robot xmlns:xacro="http://www.ros.org/wiki/xacro">
-  <xacro:macro name="warehouse_agv_gazebo" params="robot_name namespace">
+  <xacro:macro name="warehouse_agv_gazebo" params="robot_name namespace publish_odom_tf">
     <gazebo>
       <selfCollide>false</selfCollide>
@@ -20,9 +20,15 @@
         <odometryTopic>odom</odometryTopic>
         <odometryFrame>odom</odometryFrame>
-        <odometrySource>world</odometrySource>
+        <!-- Use wheel joint motion for odometry.  The world source is a
+             simulator ground-truth pose and changes when the model is
+             teleported/manually dragged, which is not valid wheel odometry
+             for the map->odom correction chain. -->
+        <odometrySource>encoder</odometrySource>
         <robotBaseFrame>base_footprint</robotBaseFrame>
         <publishWheelTF>false</publishWheelTF>
         <publishWheelJointState>true</publishWheelJointState>
-        <publishOdomTF>true</publishOdomTF>
+        <!-- publishTf enables the odometry topic in gazebo_ros_diff_drive;
+             publishOdomTF independently controls its TF broadcaster. -->
+        <publishOdomTF>${publish_odom_tf}</publishOdomTF>
         <publishTf>true</publishTf>
       </plugin>

File: src/laser-tag_nav_description/urdf/robot.urdf.xacro (robot description, xacro)
@@ -3,4 +3,5 @@
   <xacro:arg name="robot_name" default="warehouse_agv"/>
   <xacro:arg name="namespace" default="/agv"/>
+  <xacro:arg name="publish_odom_tf" default="true"/>
   <xacro:arg name="chassis_length" default="0.90"/>
   <xacro:arg name="chassis_width" default="0.64"/>
@@ -184,4 +185,7 @@
     near_clip="${bottom_camera_near_clip}"
     far_clip="${bottom_camera_far_clip}"/>
-  <xacro:warehouse_agv_gazebo robot_name="${robot_name}" namespace="${namespace}"/>
+  <xacro:warehouse_agv_gazebo
+    robot_name="${robot_name}"
+    namespace="${namespace}"
+    publish_odom_tf="$(arg publish_odom_tf)"/>
 </robot>
