Commit message: 删除velodyne雷达插件

File: src/tag_nav_description/urdf/macros.xacro (robot description, xacro)
@@ -40,17 +40,4 @@
     </inertial>
   </xacro:macro>
-  <xacro:macro name="cylinder_inertial" params="mass radius length">
-    <inertial>
-      <mass value="${mass}"/>
-      <origin xyz="0 0 0" rpy="0 0 0"/>
-      <inertia
-        ixx="${mass * (3.0 * radius * radius + length * length) / 12.0}"
-        ixy="0.0"
-        ixz="0.0"
-        iyy="${mass * (3.0 * radius * radius + length * length) / 12.0}"
-        iyz="0.0"
-        izz="${0.5 * mass * radius * radius}"/>
-    </inertial>
-  </xacro:macro>
   <xacro:macro name="box_link" params="name mass x y z material gazebo_material">
     <link name="${name}">
@@ -67,25 +54,4 @@
       </collision>
       <xacro:box_inertial mass="${mass}" x="${x}" y="${y}" z="${z}"/>
-    </link>
-    <gazebo reference="${name}">
-      <material>${gazebo_material}</material>
-    </gazebo>
-  </xacro:macro>
-  <xacro:macro name="laser_base" params="name radius length mass material gazebo_material">
-    <link name="${name}">
-      <visual>
-        <origin xyz="0 0 ${length / 2.0}" rpy="0 0 0"/>
-        <geometry>
-          <cylinder radius="${radius}" length="${length}"/>
-        </geometry>
-        <material name="${material}"/>
-      </visual>
-      <collision>
-        <origin xyz="0 0 ${length / 2.0}" rpy="0 0 0"/>
-        <geometry>
-          <cylinder radius="${radius}" length="${length}"/>
-        </geometry>
-      </collision>
-      <xacro:cylinder_inertial mass="${mass}" radius="${radius}" length="${length}"/>
     </link>
     <gazebo reference="${name}">

File: src/tag_nav_description/urdf/robot.urdf.xacro (robot description, xacro)
@@ -22,7 +22,4 @@
   <xacro:arg name="bottom_camera_far_clip" default="20.0"/>
   <xacro:arg name="ground_contact_preload" default="0.002"/>
-  <xacro:arg name="velodyne_height" default="0.27"/>
-  <xacro:arg name="laser_base_radius" default="0.02"/>
-  <xacro:arg name="laser_base_mass" default="0.25"/>
   <xacro:property name="robot_name" value="$(arg robot_name)"/>
   <xacro:property name="namespace" value="$(arg namespace)"/>
@@ -45,10 +42,5 @@
   <xacro:property name="bottom_camera_far_clip" value="$(arg bottom_camera_far_clip)"/>
   <xacro:property name="ground_contact_preload" value="$(arg ground_contact_preload)"/>
-  <xacro:property name="velodyne_height" value="$(arg velodyne_height)"/>
-  <xacro:property name="laser_base_radius" value="$(arg laser_base_radius)"/>
-  <xacro:property name="laser_base_mass" value="$(arg laser_base_mass)"/>
   <xacro:property name="base_link_height" value="0.22"/>
-  <xacro:property name="platform_top_z" value="${0.145 + 0.05 / 2.0}"/>
-  <xacro:property name="laser_base_height" value="${velodyne_height - platform_top_z}"/>
   <!-- A small preload avoids ODE treating mathematically tangent contacts as airborne. -->
   <xacro:property name="wheel_center_z" value="${wheel_radius - base_link_height - ground_contact_preload}"/>
@@ -60,5 +52,4 @@
   <xacro:property name="camera_fov" value="${120.0 * pi / 180.0}"/>
   <xacro:property name="bottom_camera_mount_z" value="${-chassis_height / 2.0}"/>
-  <xacro:include filename="$(find velodyne_description)/urdf/VLP-16.urdf.xacro"/>
   <xacro:include filename="materials.xacro"/>
   <xacro:include filename="macros.xacro"/>
@@ -91,25 +82,4 @@
     <origin xyz="0 0 0.145" rpy="0 0 0"/>
   </joint>
-  <xacro:laser_base
-    name="laser_base"
-    radius="${laser_base_radius}"
-    length="${laser_base_height}"
-    mass="${laser_base_mass}"
-    material="deck_gray"
-    gazebo_material="Gazebo/Grey"/>
-  <joint name="laser_base_joint" type="fixed">
-    <parent link="base_link"/>
-    <child link="laser_base"/>
-    <origin xyz="0 0 ${platform_top_z}" rpy="0 0 0"/>
-  </joint>
-  <xacro:VLP-16
-    parent="laser_base"
-    name="velodyne"
-    topic="/velodyne_points"
-    hz="10"
-    samples="440"
-    gpu="false">
-    <origin xyz="0 0 ${laser_base_height}" rpy="0 0 0"/>
-  </xacro:VLP-16>
   <xacro:box_link
     name="front_bumper_link"
